File: Eagle Templates for SCH and BRD/Custom Templates/LB_BIT_3IN_3OUT-LARGE-v03(1_1x)-Template/LB_BIT_3IN_3OUT-LARGE-v03(1_1x).brd (EAGLE design)
At the start: 74.2 x 24.8 mm, 37 parts, among them U1 LV321SOT23-5, U2 LV321SOT23-5, U3 LV321SOT23-5, U4 LV321SOT23-5, U5 LV321SOT23-5, U6 LV321SOT23-5

Commit message: added bitlab logo and made minor changes to board templates. Updated littlebits library.
Parts:
- added U$2: (no value), LITTLEBITS:BITLAB-LOGO
Other:
- board text added: "iX Name Here"
Changed lines of the file:
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@@
 <wire x1="-24.64" y1="36.522" x2="-25.148" y2="37.03" width="0.1016" layer="146"/>
 <text x="41.4" y="12.1" size="0.8128" layer="16" font="vector" ratio="12" rot="MR90">revX</text>
+<text x="40.9" y="23.4" size="1.3" layer="21" font="vector" rot="SR270" align="center">iX Name Here</text>
 </plain>
 <attributes>
@@
 <element name="U$1" library="LITTLEBITS" package="OSHWCREDIT" value="OSHWCREDIT" x="-95.07" y="-61.94"/>
 <element name="FRAME1" library="LITTLEBITS" package="FABDWG01-OHW" value="FRAME-LETTER" x="0" y="0"/>
+<element name="U$2" library="LITTLEBITS" package="BITLAB-LOGO" value="" x="39.4" y="27.7" rot="R270"/>
 </elements>
 <signals>

Commit message: Updated templates
- Added ferrite beads
- Moved text and annotations off of Nets layer
- Minor layout changes
- Removed I/O/W prefix from reference designators
- Removed output stage components from output bits
Parts:
- removed I?C1, I?C6, I?C7: 0.1uF, LITTLEBITS:CAP-0603
- removed I?C2: 10uF, LITTLEBITS:CAP-0603
- removed I?C3, I?C4, I?C5: 1.0uF, LITTLEBITS:CAP-0603
- removed I?R1, I?R5, I?R7: 1meg, LITTLEBITS:RES-0603
- removed I?R2, I?R6, I?R8: 10K, LITTLEBITS:RES-0603
- removed I?R3, I?R4: 3K3, LITTLEBITS:RES-0603
- removed I?TVS1, I?TVS2, I?TVS3, I?TVS4, I?TVS5, I?TVS6: ESD9B5.0ST5G, LITTLEBITS:SOD-923
- added C1, C6, C7: 0.1uF, LITTLEBITS:CAP-0603
- added C2: 10uF, LITTLEBITS:CAP-0603
- added C3, C4, C5: 1.0uF, LITTLEBITS:CAP-0603
- added FB1: FERRITE-BEAD0603, LITTLEBITS:R0603
- added R1, R5, R7: 1meg, LITTLEBITS:RES-0603
- added R2, R6, R8: 10K, LITTLEBITS:RES-0603
- added R3, R4: 3K3, LITTLEBITS:RES-0603
- added TVS1, TVS2, TVS3, TVS4, TVS5, TVS6: ESD9B5.0ST5G, LITTLEBITS:SOD-923
- moved U5 28.1 mm to (-19.8, 13.9)
- moved U4 25.8 mm to (6.60, 13.8)
- moved U3 3.76 mm to (33.0, 31.5), turned to 90 degrees
- moved U6 2.76 mm to (33.0, 13.8)
- moved U2 2.56 mm to (6.60, 31.4), turned to 90 degrees
- moved U1 1.88 mm to (-19.8, 31.4), turned to 90 degrees
- renumbered W6BSF1 to BSF4, W6BSF2 to BSF2, W6BSF3 to BSF3, W6BSM1 to BSM1, W6BSM2 to BSM2, W6BSM3 to BSM3
Connections:
- removed net SIG_IN: I?R1.2, I?R2.2, I?R5.2, I?R6.2, I?R7.2, I?R8.2, I?TVS1.2, I?TVS2.2, I?TVS3.2
- new net LB_VCC: BSF2.VCC, BSF3.VCC, BSF4.VCC, BSM1.VCC1, BSM2.VCC1, BSM3.VCC1, FB1.2
- new net N$3: BSM1.SIG1, R7.2, R8.2, TVS3.2
- new net N$4: BSM2.SIG1, R5.2, R6.2, TVS2.2
- new net N$5: BSM3.SIG1, R1.2, R2.2, TVS1.2
- net GND: now also BSF2.GND, BSF3.GND, BSF4.GND, BSM1.GND1, BSM2.GND1, BSM3.GND1, C1.2, C2.2, C3.1, C4.1, C5.1, C6.2, C7.2, R1.1, R4.1, R5.1, R7.1, TVS1.1, TVS2.1, TVS3.1, TVS4.1, TVS5.1, TVS6.1; no longer I?C1.2, I?C2.2, I?C3.1, I?C4.1, I?C5.1, I?C6.2, I?C7.2, I?R1.1, I?R4.1, I?R5.1, I?R7.1, I?TVS1.1, I?TVS2.1, I?TVS3.1, I?TVS4.1, I?TVS5.1, I?TVS6.1
- net N$1: now also R2.1; no longer I?R2.1
- net N$7: now also R6.1; no longer I?R6.1
- net N$9: now also R8.1; no longer I?R8.1
- net SIG_OUT1: now also BSF4.SIG, TVS6.2; no longer I?TVS6.2
- net SIG_OUT2: now also BSF3.SIG, TVS5.2; no longer I?TVS5.2
- net SIG_OUT3: now also BSF2.SIG, TVS4.2; no longer I?TVS4.2
- net VCC: now also C1.1, C3.2, C4.2, C5.2, C6.1, C7.1, FB1.1, R3.2; no longer I?C1.1, I?C3.2, I?C4.2, I?C5.2, I?C6.1, I?C7.1, I?R3.2
- net VREF: now also C2.1, R3.1, R4.2; no longer I?C2.1, I?R3.1, I?R4.2
Routing:
- net LB_VCC: track 0.00 -> 139.0 mm
- net VCC: track 0.00 -> 102.4 mm
- net N$7: track 0.00 -> 6.26 mm
- net N$1: track 0.00 -> 6.26 mm
- net N$9: track 0.00 -> 6.20 mm
- net SIG_OUT2: track 0.00 -> 5.37 mm
- net SIG_OUT1: track 0.00 -> 5.29 mm
- net SIG_OUT3: track 0.00 -> 5.28 mm
- net N$5: track 0.00 -> 4.82 mm
- net N$4: track 0.00 -> 4.82 mm
- net N$3: track 0.00 -> 4.68 mm
- net N$8: track 0.00 -> 2.60 mm
- net N$2: track 0.00 -> 2.60 mm
- net N$6: track 0.00 -> 2.60 mm
